File: hardware/opac_c1/v1.0/opac_c1.sch (EAGLE design)
At the start: 61 parts, among them IC1 DS3231WIDE, IC2 CP2102, IC3 ATSHA204_SOIC8, IC4 MP1584, SW1 RESET

Commit message: Revision 1 of opac.c1 board.
Parts:
- added R26, R27: (no value), resistor:R-EU_R0805
Connections:
- removed net N$29: C2.1, IC2.VDD
- new net CE_NRF24: MODULE2.GPIO0, R18.2, R27.1, SW1.1
- net N$23: now also MODULE1.CE, R26.2, R27.2; no longer MODULE2.GPIO0, R18.2, SW1.1
- net N$3: now also R26.1; no longer MODULE1.CE
- net RST: now also C2.1, IC2.VDD
Changed lines of the file:
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@@
 <part name="P+7" library="SparkFun" deviceset="3.3V" device=""/>
 <part name="P+10" library="SparkFun" deviceset="3.3V" device=""/>
+<part name="R26" library="resistor" deviceset="R-EU_" device="R0805"/>
+<part name="R27" library="resistor" deviceset="R-EU_" device="R0805"/>
 </parts>
 <sheets>
@@
 <instance part="P+7" gate="G$1" x="200.66" y="167.64"/>
 <instance part="P+10" gate="G$1" x="213.36" y="109.22"/>
+<instance part="R26" gate="G$1" x="190.5" y="109.22" rot="R90"/>
+<instance part="R27" gate="G$1" x="182.88" y="116.84"/>
 </instances>
 <busses>
@@
 <segment>
 <pinref part="MODULE1" gate="G$1" pin="!CSN"/>
-<wire x1="213.36" y1="99.06" x2="210.82" y2="99.06" width="0.1524" layer="91"/>
-<wire x1="210.82" y1="99.06" x2="210.82" y2="101.6" width="0.1524" layer="91"/>
-<pinref part="MODULE1" gate="G$1" pin="CE"/>
-<wire x1="210.82" y1="101.6" x2="213.36" y2="101.6" width="0.1524" layer="91"/>
-<wire x1="210.82" y1="101.6" x2="185.42" y2="101.6" width="0.1524" layer="91"/>
-<junction x="210.82" y="101.6"/>
+<wire x1="213.36" y1="99.06" x2="193.04" y2="99.06" width="0.1524" layer="91"/>
+<wire x1="193.04" y1="99.06" x2="193.04" y2="101.6" width="0.1524" layer="91"/>
+<wire x1="193.04" y1="101.6" x2="190.5" y2="101.6" width="0.1524" layer="91"/>
 <pinref part="R11" gate="G$1" pin="1"/>
+<wire x1="190.5" y1="101.6" x2="185.42" y2="101.6" width="0.1524" layer="91"/>
 <wire x1="185.42" y1="101.6" x2="182.88" y2="101.6" width="0.1524" layer="91"/>
 <junction x="185.42" y="101.6"/>
 <pinref part="R1" gate="G$1" pin="2"/>
+<pinref part="R26" gate="G$1" pin="1"/>
+<wire x1="190.5" y1="104.14" x2="190.5" y2="101.6" width="0.1524" layer="91"/>
+<junction x="190.5" y="101.6"/>
 </segment>
 </net>
@@
 <pinref part="MODULE1" gate="G$1" pin="VCC"/>
 <wire x1="213.36" y1="106.68" x2="213.36" y2="109.22" width="0.1524" layer="91"/>
-<label x="200.66" y="106.68" size="1.778" layer="95"/>
 <pinref part="P+10" gate="G$1" pin="3.3V"/>
 </segment>
@@
 <label x="101.6" y="170.18" size="1.778" layer="95"/>
 <pinref part="IC2" gate="G$1" pin="!RST"/>
+<wire x1="60.96" y1="162.56" x2="48.26" y2="162.56" width="0.1524" layer="91"/>
+<pinref part="C2" gate="G$1" pin="1"/>
+<pinref part="IC2" gate="G$1" pin="VDD"/>
+<wire x1="48.26" y1="162.56" x2="48.26" y2="177.8" width="0.1524" layer="91"/>
+<junction x="48.26" y="162.56"/>
+<wire x1="48.26" y1="177.8" x2="99.06" y2="177.8" width="0.1524" layer="91"/>
+<wire x1="99.06" y1="177.8" x2="99.06" y2="170.18" width="0.1524" layer="91"/>
+<junction x="99.06" y="170.18"/>
 </segment>
 </net>
@@
 </segment>
 </net>
-<net name="N$23" class="0">
+<net name="CE_NRF24" class="0">
 <segment>
 <pinref part="MODULE2" gate="G$1" pin="GPIO0"/>
@@
 <wire x1="81.28" y1="30.48" x2="81.28" y2="27.94" width="0.1524" layer="91"/>
 <junction x="81.28" y="27.94"/>
+<label x="68.58" y="27.94" size="1.778" layer="95"/>
+</segment>
+<segment>
+<pinref part="R27" gate="G$1" pin="1"/>
+<wire x1="177.8" y1="116.84" x2="172.72" y2="116.84" width="0.1524" layer="91"/>
+<label x="172.72" y="116.84" size="1.778" layer="95"/>
 </segment>
 </net>
@@
 </segment>
 </net>
-<net name="N$29" class="0">
-<segment>
-<wire x1="60.96" y1="162.56" x2="48.26" y2="162.56" width="0.1524" layer="91"/>
-<pinref part="C2" gate="G$1" pin="1"/>
-<pinref part="IC2" gate="G$1" pin="VDD"/>
-</segment>
-</net>
+<net name="N$23" class="0">
+<segment>
+<pinref part="MODULE1" gate="G$1" pin="CE"/>
+<wire x1="213.36" y1="101.6" x2="195.58" y2="101.6" width="0.1524" layer="91"/>
+<wire x1="195.58" y1="101.6" x2="195.58" y2="116.84" width="0.1524" layer="91"/>
+<wire x1="195.58" y1="116.84" x2="190.5" y2="116.84" width="0.1524" layer="91"/>
+<pinref part="R27" gate="G$1" pin="2"/>
+<pinref part="R26" gate="G$1" pin="2"/>
+<wire x1="190.5" y1="116.84" x2="187.96" y2="116.84" width="0.1524" layer="91"/>
+<wire x1="190.5" y1="114.3" x2="190.5" y2="116.84" width="0.1524" layer="91"/>
+<junction x="190.5" y="116.84"/>
+</segment>
+</net>

Commit message: Opaq.c1 revision 2.
Parts:
- added GND0: (no value), wirepad:SMD2
- C4: device resistor:C-EUC0805K -> resistor:C-EUC0603K
- renumbered VCC to 5V
Connections:
- net GND: now also GND0.P

Commit message: Opaq C1 hardware revision 3.
Parts:
- removed R24: (no value), resistor:R-EU_R0603
- removed R3, R4, R5, R6: (no value), resistor:R-EU_R0805
- added ADC: (no value), wirepad:SMD2
- added JP2, JP3: FIDUCIAL1X2.5, SparkFun:FIDUCIAL1X2.5
- added Q1: MMBT2222A, SparkFun-DiscreteSemi:TRANSISTOR_NPNMMBT2222A
- C8, C9: device resistor:C-EUC0603 -> resistor:C-EUC3216
- R2: device resistor:R-EU_R0805 -> resistor:R-EU_R0603
- SW1: value RESET -> PROG
- renumbered CE to GPIO16
Connections:
- removed net N$5: MODULE1.MOSI, R3.2
- removed net N$6: MODULE1.MISO, R4.2
- removed net SCL_C_A: IC1.SCL, R5.1, SCL.P
- removed net SDA_C_A: IC1.SDA, R6.1, SDA.P
- new net ADC_IN: ADC.P, MODULE2.ADC
- net 3.3V: now also R2.1
- net GND: now also Q1.E; no longer R24.1
- net MISO_NRF24: now also MODULE1.MISO; no longer R4.1
- net MOSI_NRF24: now also MODULE1.MOSI; no longer R3.1
- net N$19: now also Q1.C
- net N$32: no longer R24.2
- net N$4: now also C2.1, IC2.VDD; no longer MODULE1.SCK, R2.2
- net RST: now also R2.2; no longer C2.1, IC2.VDD
- net SCK_NRF24: now also MODULE1.SCK; no longer R2.1
- net SCL_C: now also IC1.SCL, SCL.P; no longer R5.2
- net SDA_C: now also IC1.SDA, SDA.P; no longer R6.2
- net SIGNAL433: now also Q1.B; no longer R8.1
- net VCC: now also R8.1
Other:
- moved on the sheet: R2, R25, R8
