File: hardware/opac_n1/v2/opaq_n1.brd (EAGLE design)
At the start: 30.3 x 50.4 mm, 38 parts, among them IC1 RT9013-XXXB, IC2 TS5A3157, IC3 ATSHA204_SOIC8, IC4 ACS712, IC5 ADS1100, IC6 ATMega-328, IC7 AT25F512BWIDE_5.3MM, IC8 LM2594HV, Q1 IRLR3915, Q2 IRLR3915, Q3 IRLR3915, Q4 IRLR3915, SW1 RESET, X1 16 MHz

Commit message: Opaq n1 board revision 1.
Parts:
- removed SW1: RESET, MySMD:157SW
- added K1: 62101021021, Wurth_Elektronik_Electromechanic_Board_to_Board_Connectors_rev15c:62101021021
- moved X1 0.64 mm to (12.4, 14.8), turned to 90 degrees
Connections:
- net A4_SDA: now also K1.10
- net A5_SCL: now also K1.9
- net D0_RX: now also K1.1
- net D11_MOSI: now also K1.7
- net D12_MISO: now also K1.3
- net D13_SCK: now also K1.4
- net D1_TX: now also K1.2
- net GND: now also K1.6; no longer SW1.2
- net RST: now also K1.5; no longer SW1.1
- net VCC: now also K1.8
Routing:
- net D0_RX: track 0.00 -> 13.3 mm, vias 0 -> 1
- net A4_SDA: track 24.8 -> 36.4 mm, vias 2 -> 3
- net D1_TX: track 0.00 -> 11.3 mm, vias 0 -> 1
- net A5_SCL: track 24.2 -> 34.7 mm, vias 0 -> 1
- net +5V: track 105.3 -> 111.9 mm
- net D11_MOSI: track 29.2 -> 34.8 mm, vias 1 -> 2
- net D13_SCK: track 38.2 -> 43.1 mm, vias 3 -> 4
- net RST: track 14.7 -> 19.3 mm
- net VCC: track 36.4 -> 40.2 mm
- net D12_MISO: track 34.6 -> 37.4 mm, vias 3 -> 4
- net N$1: track 5.90 -> 3.40 mm
- net N$21: track 3.77 -> 5.95 mm
- net GND: track 3.57 -> 3.56 mm, vias 62 -> 63

Commit message: Opaq n1 hardware revision 2.
Parts:
- added JP1, JP2: FIDUCIAL1X2.5, SparkFun:FIDUCIAL-1X2.5
- added R6, R7, R8, R9: (no value), resistor:0805
Connections:
- new net N$30: Q1.1, R6.1
- new net N$31: Q3.1, R7.1
- new net N$32: Q2.1, R8.1
- new net N$33: Q4.1, R9.1
- net DIM1: now also R6.2; no longer Q1.1
- net DIM2: now also R8.2; no longer Q2.1
- net DIM3: now also R7.2; no longer Q3.1
- net DIM4: now also R9.2; no longer Q4.1
Routing:
- net DIM1: track 47.1 -> 23.9 mm, vias 2 -> 0
- net N$30: track 0.00 -> 21.9 mm, vias 0 -> 2
- net DIM2: track 41.6 -> 26.3 mm
- net N$32: track 0.00 -> 14.2 mm
- net DIM3: track 40.8 -> 37.1 mm
- net N$33: track 0.00 -> 2.55 mm
- net DIM4: track 30.3 -> 27.9 mm
- net N$31: track 0.00 -> 2.14 mm
