File: hardware/opac_n1/v2/opaq_n1.sch (EAGLE design)
At the start: 38 parts, among them IC1 RT9013-XXXB, IC2 TS5A3157, IC3 ATSHA204_SOIC8, IC4 ACS712, IC5 ADS1100, IC6 ATMega-328, IC7 AT25F512BWIDE_5.3MM, IC8 LM2594HV, Q1 IRLR3915, Q2 IRLR3915, Q3 IRLR3915, Q4 IRLR3915, SW1 RESET, X1 16 MHz

Commit message: Opaq n1 board revision 1.
Parts:
- removed SW1: RESET, MySMD:PB157
- added K1: 62101021021, Wurth_Elektronik_Electromechanic_Board_to_Board_Connectors_rev15c:62101021021
Connections:
- net A4_SDA: now also K1.10
- net A5_SCL: now also K1.9
- net D0_RX: now also K1.1
- net D11_MOSI: now also K1.7
- net D12_MISO: now also K1.3
- net D13_SCK: now also K1.4
- net D1_TX: now also K1.2
- net GND: now also K1.6; no longer SW1.2
- net RST: now also K1.5; no longer SW1.1
- net VCC: now also K1.8
Changed lines of the file:
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@@
 <part name="P+10" library="SparkFun" deviceset="3.3V" device=""/>
 <part name="GND8" library="supply1" deviceset="GND" device=""/>
-<part name="SW1" library="MySMD" deviceset="PB157" device="" value="RESET">
-<attribute name="PARTNO" value="RS 682-1421"/>
-</part>
 <part name="SUPPLY4" library="SparkFun" deviceset="VCC" device="" value="5v"/>
 <part name="SUPPLY5" library="supply2" deviceset="GND" device=""/>
@@
 <part name="P+12" library="SparkFun" deviceset="VCC" device="" value="5v"/>
 <part name="IC7" library="LowPowerLab" deviceset="AT25F512B" device="WIDE_5.3MM" value="AT25F512BWIDE_5.3MM"/>
-<part name="SUPPLY1" library="supply2" deviceset="GND" device=""/>
 <part name="C7" library="SparkFun-Passives" deviceset="CAP" device="0402-CAP" value="100pf"/>
 <part name="FRAME2" library="SparkFun-Aesthetics" deviceset="FRAME-LETTER" device="NO_PACKAGE"/>
@@
 <part name="C10" library="rcl" deviceset="CPOL-EU" device="D/7343-31R"/>
 <part name="GND11" library="SparkFun" deviceset="GND" device=""/>
+<part name="K1" library="Wurth_Elektronik_Electromechanic_Board_to_Board_Connectors_rev15c" deviceset="62101021021" device=""/>
+<part name="GND15" library="SparkFun-Aesthetics" deviceset="GND" device=""/>
 </parts>
 <sheets>
@@
 <instance part="P+10" gate="G$1" x="170.18" y="96.52"/>
 <instance part="GND8" gate="1" x="165.1" y="91.44" rot="R180"/>
-<instance part="SW1" gate="G$1" x="53.34" y="129.54">
-<attribute name="PARTNO" x="53.34" y="129.54" size="1.778" layer="96" display="off"/>
-</instance>
 <instance part="SUPPLY4" gate="1" x="31.75" y="124.46"/>
 <instance part="SUPPLY5" gate="GND" x="31.75" y="86.36"/>
@@
 <attribute name="VALUE" x="121.92" y="49.022" size="1.778" layer="96" rot="R180"/>
 </instance>
-<instance part="SUPPLY1" gate="GND" x="60.96" y="124.46"/>
 <instance part="R1" gate="G$1" x="139.7" y="116.84" rot="R90"/>
 <instance part="R5" gate="G$1" x="147.32" y="127" rot="R180"/>
@@
 <instance part="C10" gate="G$1" x="96.52" y="165.1"/>
 <instance part="GND11" gate="1" x="96.52" y="152.4"/>
+<instance part="K1" gate="G$1" x="81.28" y="22.86"/>
+<instance part="GND15" gate="1" x="93.98" y="17.78"/>
 </instances>
 <busses>
@@
 </segment>
 <segment>
-<pinref part="SUPPLY1" gate="GND" pin="GND"/>
-<pinref part="SW1" gate="G$1" pin="2"/>
-<wire x1="60.96" y1="127" x2="60.96" y2="129.54" width="0.1524" layer="91"/>
-</segment>
-<segment>
 <pinref part="R1" gate="G$1" pin="1"/>
 <pinref part="GND13" gate="1" pin="GND"/>
@@
 <pinref part="C10" gate="G$1" pin="-"/>
 <wire x1="96.52" y1="154.94" x2="96.52" y2="160.02" width="0.1524" layer="91"/>
+</segment>
+<segment>
+<pinref part="K1" gate="G$1" pin="6"/>
+<pinref part="GND15" gate="1" pin="GND"/>
+<wire x1="86.36" y1="22.86" x2="93.98" y2="22.86" width="0.1524" layer="91"/>
+<wire x1="93.98" y1="22.86" x2="93.98" y2="20.32" width="0.1524" layer="91"/>
 </segment>
 </net>
@@
 <net name="RST" class="0">
 <segment>
-<label x="42.926" y="109.728" size="1.778" layer="95"/>
+<label x="40.386" y="112.268" size="1.778" layer="95"/>
 <pinref part="IC6" gate="G$1" pin="PC6(/RESET)"/>
-<wire x1="41.91" y1="111.76" x2="43.18" y2="111.76" width="0.1524" layer="91"/>
 <pinref part="R2" gate="G$1" pin="2"/>
-<wire x1="43.18" y1="111.76" x2="44.45" y2="111.76" width="0.1524" layer="91"/>
-<wire x1="43.18" y1="111.76" x2="43.18" y2="129.54" width="0.1524" layer="91"/>
-<junction x="43.18" y="111.76"/>
-<pinref part="SW1" gate="G$1" pin="1"/>
-<wire x1="43.18" y1="129.54" x2="45.72" y2="129.54" width="0.1524" layer="91"/>
+<wire x1="41.91" y1="111.76" x2="44.45" y2="111.76" width="0.1524" layer="91"/>
+</segment>
+<segment>
+<pinref part="K1" gate="G$1" pin="5"/>
+<wire x1="73.66" y1="22.86" x2="63.5" y2="22.86" width="0.1524" layer="91"/>
+<label x="66.04" y="22.86" size="1.778" layer="95"/>
 </segment>
 </net>
@@
 <junction x="31.75" y="111.76"/>
 </segment>
+<segment>
+<pinref part="K1" gate="G$1" pin="8"/>
+<wire x1="86.36" y1="27.94" x2="99.06" y2="27.94" width="0.1524" layer="91"/>
+<label x="88.9" y="27.94" size="1.778" layer="95"/>
+</segment>
 </net>
 <net name="D8" class="0">
@@
 <pinref part="IC6" gate="G$1" pin="PD1(TXD)"/>
 </segment>
+<segment>
+<pinref part="K1" gate="G$1" pin="2"/>
+<wire x1="73.66" y1="30.48" x2="63.5" y2="30.48" width="0.1524" layer="91"/>
+<label x="66.04" y="30.48" size="1.778" layer="95"/>
+</segment>
 </net>
 <net name="D0_RX" class="0">
@@
 <label x="95.25" y="88.9" size="1.778" layer="95"/>
 <pinref part="IC6" gate="G$1" pin="PD0(RXD)"/>
+</segment>
+<segment>
+<pinref part="K1" gate="G$1" pin="1"/>
+<wire x1="73.66" y1="33.02" x2="63.5" y2="33.02" width="0.1524" layer="91"/>
+<label x="66.04" y="33.02" size="1.778" layer="95"/>
 </segment>
 </net>
@@
 <pinref part="R16" gate="G$1" pin="1"/>
 </segment>
+<segment>
+<pinref part="K1" gate="G$1" pin="10"/>
+<wire x1="86.36" y1="33.02" x2="99.06" y2="33.02" width="0.1524" layer="91"/>
+<label x="88.9" y="33.02" size="1.778" layer="95"/>
+</segment>
 </net>
 <net name="A3" class="0">
@@
 <label x="160.02" y="78.74" size="1.778" layer="95"/>
 </segment>
+<segment>
+<pinref part="K1" gate="G$1" pin="7"/>
+<wire x1="86.36" y1="25.4" x2="99.06" y2="25.4" width="0.1524" layer="91"/>
+<label x="88.9" y="25.4" size="1.778" layer="95"/>
+</segment>
 </net>
 <net name="D12_MISO" class="0">
@@
 <label x="160.02" y="76.2" size="1.778" layer="95"/>
 </segment>
+<segment>
+<pinref part="K1" gate="G$1" pin="3"/>
+<wire x1="73.66" y1="27.94" x2="63.5" y2="27.94" width="0.1524" layer="91"/>
+<label x="66.04" y="27.94" size="1.778" layer="95"/>
+</segment>
 </net>
 <net name="D13_SCK" class="0">
@@
 <wire x1="175.26" y1="81.28" x2="157.48" y2="81.28" width="0.1524" layer="91"/>
 <label x="160.02" y="81.28" size="1.778" layer="95"/>
+</segment>
+<segment>
+<pinref part="K1" gate="G$1" pin="4"/>
+<wire x1="73.66" y1="25.4" x2="63.5" y2="25.4" width="0.1524" layer="91"/>
+<label x="66.04" y="25.4" size="1.778" layer="95"/>
 </segment>
 </net>
@@
 <pinref part="R17" gate="G$1" pin="1"/>
 </segment>
-</net>
+<segment>
+<pinref part="K1" gate="G$1" pin="9"/>
+<wire x1="86.36" y1="30.48" x2="99.06" y2="30.48" width="0.1524" layer="91"/>
+<label x="88.9" y="30.48" size="1.778" layer="95"/>
+</segment>
+</net>

Commit message: Opaq n1 hardware revision 2.
Parts:
- added JP1, JP2: FIDUCIAL1X2.5, SparkFun:FIDUCIAL1X2.5
- added R6, R7, R8, R9: (no value), resistor:R-EU_R0805
Connections:
- new net N$30: Q1.G, R6.1
- new net N$31: Q3.G, R7.1
- new net N$32: Q2.G, R8.1
- new net N$33: Q4.G, R9.1
- net DIM1: now also R6.2; no longer Q1.G
- net DIM2: now also R8.2; no longer Q2.G
- net DIM3: now also R7.2; no longer Q3.G
- net DIM4: now also R9.2; no longer Q4.G
Changed lines of the file:
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@@
 <part name="K1" library="Wurth_Elektronik_Electromechanic_Board_to_Board_Connectors_rev15c" deviceset="62101021021" device=""/>
 <part name="GND15" library="SparkFun-Aesthetics" deviceset="GND" device=""/>
+<part name="JP1" library="SparkFun" deviceset="FIDUCIAL" device="1X2.5"/>
+<part name="JP2" library="SparkFun" deviceset="FIDUCIAL" device="1X2.5"/>
+<part name="R6" library="resistor" deviceset="R-EU_" device="R0805"/>
+<part name="R7" library="resistor" deviceset="R-EU_" device="R0805"/>
+<part name="R8" library="resistor" deviceset="R-EU_" device="R0805"/>
+<part name="R9" library="resistor" deviceset="R-EU_" device="R0805"/>
 </parts>
 <sheets>
@@
 <instance part="K1" gate="G$1" x="81.28" y="22.86"/>
 <instance part="GND15" gate="1" x="93.98" y="17.78"/>
+<instance part="JP1" gate="G$1" x="142.24" y="25.4"/>
+<instance part="JP2" gate="G$1" x="142.24" y="20.32"/>
 </instances>
 <busses>
@@
 <attribute name="NAME" x="63.246" y="113.538" size="1.778" layer="95" rot="R180"/>
 </instance>
+<instance part="R6" gate="G$1" x="137.16" y="91.44" rot="R180"/>
+<instance part="R7" gate="G$1" x="129.54" y="66.04" rot="R180"/>
+<instance part="R8" gate="G$1" x="172.72" y="91.44" rot="R180"/>
+<instance part="R9" gate="G$1" x="172.72" y="66.04" rot="R180"/>
 </instances>
 <busses>
@@
 <net name="DIM1" class="0">
 <segment>
-<pinref part="Q1" gate="G$1" pin="G"/>
-<wire x1="152.4" y1="91.44" x2="142.24" y2="91.44" width="0.1524" layer="91"/>
-<label x="144.78" y="91.44" size="1.778" layer="95"/>
+<pinref part="R6" gate="G$1" pin="2"/>
+<wire x1="132.08" y1="91.44" x2="114.3" y2="91.44" width="0.1524" layer="91"/>
+<label x="124.46" y="91.44" size="1.778" layer="95"/>
 </segment>
 </net>
 <net name="DIM2" class="0">
 <segment>
-<pinref part="Q2" gate="G$1" pin="G"/>
-<wire x1="187.96" y1="91.44" x2="177.8" y2="91.44" width="0.1524" layer="91"/>
-<label x="180.34" y="91.44" size="1.778" layer="95"/>
+<pinref part="R8" gate="G$1" pin="2"/>
+<wire x1="167.64" y1="91.44" x2="162.56" y2="91.44" width="0.1524" layer="91"/>
+<label x="162.56" y="91.44" size="1.778" layer="95"/>
 </segment>
 </net>
 <net name="DIM3" class="0">
 <segment>
-<pinref part="Q3" gate="G$1" pin="G"/>
-<wire x1="152.4" y1="66.04" x2="134.62" y2="66.04" width="0.1524" layer="91"/>
-<label x="137.16" y="66.04" size="1.778" layer="95"/>
+<pinref part="R7" gate="G$1" pin="2"/>
+<wire x1="124.46" y1="66.04" x2="111.76" y2="66.04" width="0.1524" layer="91"/>
+<label x="119.38" y="66.04" size="1.778" layer="95"/>
 </segment>
 </net>
 <net name="DIM4" class="0">
 <segment>
-<pinref part="Q4" gate="G$1" pin="G"/>
-<wire x1="187.96" y1="66.04" x2="177.8" y2="66.04" width="0.1524" layer="91"/>
-<label x="180.34" y="66.04" size="1.778" layer="95"/>
+<pinref part="R9" gate="G$1" pin="2"/>
+<wire x1="167.64" y1="66.04" x2="162.56" y2="66.04" width="0.1524" layer="91"/>
+<label x="162.56" y="66.04" size="1.778" layer="95"/>
 </segment>
 </net>
@@
 </segment>
 </net>
+<net name="N$30" class="0">
+<segment>
+<pinref part="Q1" gate="G$1" pin="G"/>
+<wire x1="152.4" y1="91.44" x2="142.24" y2="91.44" width="0.1524" layer="91"/>
+<label x="144.78" y="91.44" size="1.778" layer="95"/>
+<pinref part="R6" gate="G$1" pin="1"/>
+</segment>
+</net>
+<net name="N$31" class="0">
+<segment>
+<pinref part="Q3" gate="G$1" pin="G"/>
+<wire x1="152.4" y1="66.04" x2="134.62" y2="66.04" width="0.1524" layer="91"/>
+<label x="137.16" y="66.04" size="1.778" layer="95"/>
+<pinref part="R7" gate="G$1" pin="1"/>
+</segment>
+</net>
+<net name="N$32" class="0">
+<segment>
+<pinref part="Q2" gate="G$1" pin="G"/>
+<wire x1="187.96" y1="91.44" x2="177.8" y2="91.44" width="0.1524" layer="91"/>
+<label x="180.34" y="91.44" size="1.778" layer="95"/>
+<pinref part="R8" gate="G$1" pin="1"/>
+</segment>
+</net>
+<net name="N$33" class="0">
+<segment>
+<pinref part="Q4" gate="G$1" pin="G"/>
+<wire x1="187.96" y1="66.04" x2="177.8" y2="66.04" width="0.1524" layer="91"/>
+<label x="180.34" y="66.04" size="1.778" layer="95"/>
+<pinref part="R9" gate="G$1" pin="1"/>
+</segment>
+</net>
