File: hardware/opac_c1/v1.1/opac_c1.sch (EAGLE design)
At the start: 77 parts, among them IC2 CP2102, IC3 ATSHA204_SOIC8, IC4 MP1584, IC5 TSC2046QFN, IC6 ATMega-328, IC7 RT9300, IC8 DS1307SO8, Q1 MMBT2222A, Q2 32.768kHz mc306, SW1 PROG, X1 8 MHz

Commit message: Updated version of the opaq c1 hardware.
Parts:
- C10, C13, C7: value (none) -> 0.1uf
- C4: value (none) -> 47nH
- C8, C9: value (none) -> 10uf
- D1: value (none) -> SS34
- L1: value (none) -> 4.7uh
- R20: value (none) -> 8.2k
- R21: value (none) -> 24k
- R22, R23, R25: value (none) -> 100k
Changed lines of the file:
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@@
 </part>
 <part name="R13" library="resistor" deviceset="R-EU_" device="R0603"/>
-<part name="C4" library="resistor" deviceset="C-EU" device="C0603K"/>
+<part name="C4" library="resistor" deviceset="C-EU" device="C0603K" value="47nH"/>
 <part name="P+3" library="SparkFun" deviceset="3.3V" device=""/>
 <part name="GPIO16" library="wirepad" deviceset="SMD2" device=""/>
@@
 <part name="P+2" library="SparkFun" deviceset="VCC" device=""/>
 <part name="GND11" library="SparkFun" deviceset="GND" device=""/>
-<part name="D1" library="SparkFun" deviceset="DIODE" device="SMA"/>
-<part name="L1" library="RNH_IHLP-2525CZ-01" deviceset="IHLP-2525CZ-01" device=""/>
+<part name="D1" library="SparkFun" deviceset="DIODE" device="SMA" value="SS34"/>
+<part name="L1" library="RNH_IHLP-2525CZ-01" deviceset="IHLP-2525CZ-01" device="" value="4.7uh"/>
 <part name="GND13" library="SparkFun" deviceset="GND" device=""/>
-<part name="C7" library="resistor" deviceset="C-EU" device="C0603"/>
-<part name="C8" library="resistor" deviceset="C-EU" device="C3216"/>
+<part name="C7" library="resistor" deviceset="C-EU" device="C0603" value="0.1uf"/>
+<part name="C8" library="resistor" deviceset="C-EU" device="C3216" value="10uf"/>
 <part name="GND14" library="SparkFun" deviceset="GND" device=""/>
-<part name="R20" library="resistor" deviceset="R-EU_" device="R0603"/>
-<part name="R21" library="resistor" deviceset="R-EU_" device="R0603"/>
+<part name="R20" library="resistor" deviceset="R-EU_" device="R0603" value="8.2k"/>
+<part name="R21" library="resistor" deviceset="R-EU_" device="R0603" value="24k"/>
 <part name="GND15" library="SparkFun" deviceset="GND" device=""/>
-<part name="C9" library="resistor" deviceset="C-EU" device="C3216"/>
-<part name="C10" library="resistor" deviceset="C-EU" device="C0603"/>
+<part name="C9" library="resistor" deviceset="C-EU" device="C3216" value="10uf"/>
+<part name="C10" library="resistor" deviceset="C-EU" device="C0603" value="0.1uf"/>
 <part name="C11" library="resistor" deviceset="C-EU" device="C0603"/>
-<part name="R22" library="resistor" deviceset="R-EU_" device="R0603"/>
-<part name="R23" library="resistor" deviceset="R-EU_" device="R0603"/>
+<part name="R22" library="resistor" deviceset="R-EU_" device="R0603" value="100k"/>
+<part name="R23" library="resistor" deviceset="R-EU_" device="R0603" value="100k"/>
 <part name="GND16" library="SparkFun" deviceset="GND" device=""/>
-<part name="R25" library="resistor" deviceset="R-EU_" device="R0603"/>
+<part name="R25" library="resistor" deviceset="R-EU_" device="R0603" value="100k"/>
 <part name="GND18" library="SparkFun" deviceset="GND" device=""/>
 <part name="GND19" library="SparkFun" deviceset="GND" device=""/>
@@
 <part name="GPIO5" library="wirepad" deviceset="SMD2" device=""/>
 <part name="P+15" library="SparkFun" deviceset="3.3V" device=""/>
-<part name="C13" library="resistor" deviceset="C-EU" device="C0603"/>
+<part name="C13" library="resistor" deviceset="C-EU" device="C0603" value="0.1uf"/>
 <part name="P+17" library="SparkFun" deviceset="VCC" device=""/>
 <part name="P+18" library="SparkFun" deviceset="3.3V" device=""/>
