File: hardware/n1/v2.1/opaq_n1.brd (EAGLE design)
At the start: 30.3 x 50.4 mm, 44 parts, among them IC1 RT9013-XXXB, IC2 TS5A3157, IC3 ATSHA204_SOIC8, IC4 ACS712, IC5 ADS1100, IC6 ATMega-328, IC7 AT25F512BWIDE_5.3MM, IC8 LM2594HV, K1 62101021021, Q1 IRLR3915, Q2 IRLR3915, Q3 IRLR3915, Q4 IRLR3915, X1 16 MHz

Commit message: Updated the Opaq n1 firmware to read the external temperature and the input voltage. Added the support for the external flash. Renamed the folder of the Opaq n1 hardware.
Parts:
- R1: value (none) -> 1.62k
- R5: value (none) -> 28k
Changed lines of the file:
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@@
 <attribute name="DESIGNER" value="Nobody" x="-19.5072" y="-10.1214" size="1.778" layer="27" display="off"/>
 </element>
-<element name="R1" library="resistor" package="0805" value="" x="26.9" y="8.5" smashed="yes" rot="R180">
+<element name="R1" library="resistor" package="0805" value="1.62k" x="26.9" y="8.5" smashed="yes" rot="R180">
 <attribute name="NAME" x="25.635078125" y="8.7413" size="0.6096" layer="25" ratio="14" rot="R180"/>
 <attribute name="VALUE" x="27.916" y="9.897" size="0.4064" layer="27" rot="R180"/>
 </element>
-<element name="R5" library="resistor" package="0805" value="" x="26.9" y="11.2" smashed="yes" rot="R180">
+<element name="R5" library="resistor" package="0805" value="28k" x="26.9" y="11.2" smashed="yes" rot="R180">
 <attribute name="NAME" x="25.599521875" y="11.4413" size="0.6096" layer="25" ratio="14" rot="R180"/>
 <attribute name="VALUE" x="27.916" y="12.597" size="0.4064" layer="27" rot="R180"/>
